File: pcb/code40.kicad_pcb (KiCad board)
At the start: 2 copper layers, 229 x 105 mm, 101 parts, among them K1 KEYSW, K10 KEYSW, K11 KEYSW, K12 KEYSW, K13 KEYSW, K14 KEYSW, K15 KEYSW, K16 KEYSW, K17 KEYSW, K18 KEYSW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

Commit message: new kicad version
Other:
- net class Default removed
